Commit message: 3d建图

File: mycar/src/mycar_f/urdf/mycar_f.urdf (robot description, URDF)
Before this commit: robot mycar_f, 8 links, 7 joints
Joints:
- joint base_footprint_joint: origin xyz=0 0 0 rpy=0 0 0 -> xyz=0 0 0.066 rpy=0 0 0
- joint camera_joint: origin xyz=0.0936947862405823 -0.0316811986946451 0.0440937058350375 rpy=3.14159 0 0 -> xyz=0.0936947862405823 -0.0316811986946451 0.0440937058350375 rpy=0 0 0
